File: pico-power-board.kicad_sch (KiCad schematic)
At the start: 109 parts, among them J1 Conn_02x10_Counter_Clockwise, J10 Conn_01x20_Female, J2 Conn_02x10_Counter_Clockwise, J3 Conn_02x10_Counter_Clockwise, J4 Conn_02x10_Counter_Clockwise, J5 Conn_02x10_Counter_Clockwise, J6 Conn_02x10_Counter_Clockwise, J7 DC-042C-Z-2.5, J8 Conn_01x06_Male, J9 Conn_01x20_Female, U1 TMP112AIDRLR, U2 INA219AxD, U3 K7803-500R3, U4 74LVC1G125GW,125, U5 74LVC1G125GW,125, U6 74LVC1G125GW,125, U7 74LVC1G125GW,125, U8 74LVC1G125GW,125, U9 74LVC1G125GW,125

Commit message: Revision v0.1
Parts:
- R13, R15, R17, R31, R33, R35: value 30k -> 27k; LCSC C22984 -> C308131
- U3: LCSC C909766 -> C86736
Other:
- note added: "TODO: - does voltage divider on reset line or pull ups on chip-select affect termination and voltage level? -> we'll see - check inner diameter of barrel jack (2.1 or 2.5mm) -> 2.5mm - DC Jack and Female Headers often out of stock at JLCPCB -> maybe pre-order those parts -> just use different parts that are in stock"
- note removed: "TODO: - does voltage divider on reset line or pull ups on chip-select affect termination and voltage level? - check inner diameter of barrel jack (2.1 or 2.5mm) -> probably 2.5mm - DC Jack and Female Headers often out of stock at JLCPCB - maybe pre-order those parts"
Changed lines of the file:
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@@
     (effects (font (size 1.27 1.27)) (justify left bottom))
   )
-  (text "TODO:\n\n- does voltage divider on reset line or pull ups on chip-select affect termination and voltage level?\n\n- check inner diameter of barrel jack (2.1 or 2.5mm) -> probably 2.5mm\n- DC Jack and Female Headers often out of stock at JLCPCB\n	- maybe pre-order those parts"
-    (at 26.67 262.89 0)
+  (text "TODO:\n\n- does voltage divider on reset line or pull ups on chip-select affect termination and voltage level?\n	-> we'll see\n\n- check inner diameter of barrel jack (2.1 or 2.5mm)\n	-> 2.5mm\n- DC Jack and Female Headers often out of stock at JLCPCB\n	-> maybe pre-order those parts\n	-> just use different parts that are in stock"
+    (at 22.86 254 0)
     (effects (font (size 1.27 1.27)) (justify left bottom))
   )
@@
       (effects (font (size 1.27 1.27)) (justify left))
     )
-    (property "Value" "30k" (at 72.39 92.71 0)
+    (property "Value" "27k" (at 72.39 92.71 0)
       (effects (font (size 1.27 1.27)) (justify left))
     )
@@
       (effects (font (size 1.27 1.27)) hide)
     )
-    (property "Datasheet" "https://datasheet.lcsc.com/lcsc/2206010116_UNI-ROYAL-Uniroyal-Elec-0603WAF3002T5E_C22984.pdf" (at 73.66 93.98 0)
+    (property "Datasheet" "https://datasheet.lcsc.com/lcsc/2304140030_ROHM-Semicon-MCR03ERTJ273_C308131.pdf" (at 73.66 93.98 0)
       (effects (font (size 1.27 1.27)) hide)
     )
-    (property "LCSC" "C22984" (at 73.66 93.98 0)
+    (property "LCSC" "C308131" (at 73.66 93.98 0)
       (effects (font (size 1.27 1.27)) hide)
     )
@@
       (effects (font (size 1.27 1.27) italic) hide)
     )
-    (property "Datasheet" "https://item.szlcsc.com/421835.html" (at 352.044 83.693 0)
+    (property "Datasheet" "https://jlcpcb.com/b63bad90-f7ef-4c31-9399-51c6d3152fc3" (at 352.044 83.693 0)
       (effects (font (size 1.27 1.27)) (justify left) hide)
     )
@@
       (effects (font (size 1.27 1.27) italic) hide)
     )
-    (property "Datasheet" "https://item.szlcsc.com/421835.html" (at 352.044 182.753 0)
+    (property "Datasheet" "https://jlcpcb.com/b63bad90-f7ef-4c31-9399-51c6d3152fc3" (at 352.044 182.753 0)
       (effects (font (size 1.27 1.27)) (justify left) hide)
     )
@@
       (effects (font (size 1.27 1.27) italic) hide)
     )
-    (property "Datasheet" "https://item.szlcsc.com/421835.html" (at 352.044 116.713 0)
+    (property "Datasheet" "https://jlcpcb.com/b63bad90-f7ef-4c31-9399-51c6d3152fc3" (at 352.044 116.713 0)
       (effects (font (size 1.27 1.27)) (justify left) hide)
     )
@@
       (effects (font (size 1.27 1.27) italic) hide)
     )
-    (property "Datasheet" "https://item.szlcsc.com/421835.html" (at 352.044 149.733 0)
+    (property "Datasheet" "https://jlcpcb.com/b63bad90-f7ef-4c31-9399-51c6d3152fc3" (at 352.044 149.733 0)
       (effects (font (size 1.27 1.27)) (justify left) hide)
     )
@@
       (effects (font (size 1.27 1.27)) hide)
     )
-    (property "Value" "+3V3" (at 360.68 143.51 0)
+    (property "Value" "+3V3" (at 364.49 140.97 0)
       (effects (font (size 1.27 1.27)))
     )
@@
       (effects (font (size 1.27 1.27)) (justify left))
     )
-    (property "Value" "30k" (at 129.54 92.71 0)
+    (property "Value" "27k" (at 129.54 92.71 0)
       (effects (font (size 1.27 1.27)) (justify left))
     )
@@
       (effects (font (size 1.27 1.27)) hide)
     )
-    (property "Datasheet" "https://datasheet.lcsc.com/lcsc/2206010116_UNI-ROYAL-Uniroyal-Elec-0603WAF3002T5E_C22984.pdf" (at 130.81 93.98 0)
+    (property "Datasheet" "https://datasheet.lcsc.com/lcsc/2304140030_ROHM-Semicon-MCR03ERTJ273_C308131.pdf" (at 130.81 93.98 0)
       (effects (font (size 1.27 1.27)) hide)
     )
-    (property "LCSC" "C22984" (at 130.81 93.98 0)
+    (property "LCSC" "C308131" (at 130.81 93.98 0)
       (effects (font (size 1.27 1.27)) hide)
     )
@@
       (effects (font (size 1.27 1.27) italic) hide)
     )
-    (property "Datasheet" "https://item.szlcsc.com/421835.html" (at 352.044 49.403 0)
+    (property "Datasheet" "https://jlcpcb.com/b63bad90-f7ef-4c31-9399-51c6d3152fc3" (at 352.044 49.403 0)
       (effects (font (size 1.27 1.27)) (justify left) hide)
     )
@@
       (effects (font (size 1.27 1.27)) (justify left))
     )
-    (property "Value" "30k" (at 129.54 138.43 0)
+    (property "Value" "27k" (at 129.54 138.43 0)
       (effects (font (size 1.27 1.27)) (justify left))
     )
@@
       (effects (font (size 1.27 1.27)) hide)
     )
-    (property "Datasheet" "https://datasheet.lcsc.com/lcsc/2206010116_UNI-ROYAL-Uniroyal-Elec-0603WAF3002T5E_C22984.pdf" (at 130.81 139.7 0)
+    (property "Datasheet" "https://datasheet.lcsc.com/lcsc/2304140030_ROHM-Semicon-MCR03ERTJ273_C308131.pdf" (at 130.81 139.7 0)
       (effects (font (size 1.27 1.27)) hide)
     )
-    (property "LCSC" "C22984" (at 130.81 139.7 0)
+    (property "LCSC" "C308131" (at 130.81 139.7 0)
       (effects (font (size 1.27 1.27)) hide)
     )
@@
       (effects (font (size 1.27 1.27)) (justify left))
     )
-    (property "Value" "30k" (at 129.54 46.99 0)
+    (property "Value" "27k" (at 129.54 46.99 0)
       (effects (font (size 1.27 1.27)) (justify left))
     )
@@
       (effects (font (size 1.27 1.27)) hide)
     )
-    (property "Datasheet" "https://datasheet.lcsc.com/lcsc/2206010116_UNI-ROYAL-Uniroyal-Elec-0603WAF3002T5E_C22984.pdf" (at 130.81 48.26 0)
+    (property "Datasheet" "https://datasheet.lcsc.com/lcsc/2304140030_ROHM-Semicon-MCR03ERTJ273_C308131.pdf" (at 130.81 48.26 0)
       (effects (font (size 1.27 1.27)) hide)
     )
-    (property "LCSC" "C22984" (at 130.81 48.26 0)
+    (property "LCSC" "C308131" (at 130.81 48.26 0)
       (effects (font (size 1.27 1.27)) hide)
     )
@@
       (effects (font (size 1.27 1.27)) hide)
     )
-    (property "Value" "+3V3" (at 360.68 77.47 0)
+    (property "Value" "+3V3" (at 364.49 74.93 0)
       (effects (font (size 1.27 1.27)))
     )
@@
       (effects (font (size 1.27 1.27) italic) hide)
     )
-    (property "Datasheet" "https://datasheet.lcsc.com/lcsc/2011180207_DEXU-Electronics-K7803-500R3_C909766.pdf" (at 274.32 198.12 0)
+    (property "Datasheet" "https://www.mornsun-power.com/html/pdf/K7803-500R3.html" (at 274.32 198.12 0)
       (effects (font (size 1.27 1.27)) (justify left) hide)
     )
-    (property "LCSC" "C909766" (at 269.24 181.61 0)
+    (property "LCSC" "C86736" (at 269.24 181.61 0)
       (effects (font (size 1.27 1.27)) hide)
     )
@@
       (effects (font (size 1.27 1.27)) (justify left))
     )
-    (property "Value" "30k" (at 72.39 46.99 0)
+    (property "Value" "27k" (at 72.39 46.99 0)
       (effects (font (size 1.27 1.27)) (justify left))
     )
@@
       (effects (font (size 1.27 1.27)) hide)
     )
-    (property "Datasheet" "https://datasheet.lcsc.com/lcsc/2206010116_UNI-ROYAL-Uniroyal-Elec-0603WAF3002T5E_C22984.pdf" (at 73.66 48.26 0)
+    (property "Datasheet" "https://datasheet.lcsc.com/lcsc/2304140030_ROHM-Semicon-MCR03ERTJ273_C308131.pdf" (at 73.66 48.26 0)
       (effects (font (size 1.27 1.27)) hide)
     )
-    (property "LCSC" "C22984" (at 73.66 48.26 0)
+    (property "LCSC" "C308131" (at 73.66 48.26 0)
       (effects (font (size 1.27 1.27)) hide)
     )
@@
       (effects (font (size 1.27 1.27) italic) hide)
     )
-    (property "Datasheet" "https://item.szlcsc.com/421835.html" (at 352.044 215.773 0)
+    (property "Datasheet" "https://jlcpcb.com/b63bad90-f7ef-4c31-9399-51c6d3152fc3" (at 352.044 215.773 0)
       (effects (font (size 1.27 1.27)) (justify left) hide)
     )
@@
       (effects (font (size 1.27 1.27)) (justify left))
     )
-    (property "Value" "30k" (at 72.39 138.43 0)
+    (property "Value" "27k" (at 72.39 138.43 0)
       (effects (font (size 1.27 1.27)) (justify left))
     )
@@
       (effects (font (size 1.27 1.27)) hide)
     )
-    (property "Datasheet" "https://datasheet.lcsc.com/lcsc/2206010116_UNI-ROYAL-Uniroyal-Elec-0603WAF3002T5E_C22984.pdf" (at 73.66 139.7 0)
+    (property "Datasheet" "https://datasheet.lcsc.com/lcsc/2304140030_ROHM-Semicon-MCR03ERTJ273_C308131.pdf" (at 73.66 139.7 0)
       (effects (font (size 1.27 1.27)) hide)
     )
-    (property "LCSC" "C22984" (at 73.66 139.7 0)
+    (property "LCSC" "C308131" (at 73.66 139.7 0)
       (effects (font (size 1.27 1.27)) hide)
     )
@@
       (effects (font (size 1.27 1.27)) hide)
     )
-    (property "Value" "+3V3" (at 360.68 209.55 0)
+    (property "Value" "+3V3" (at 364.49 207.01 0)
       (effects (font (size 1.27 1.27)))
     )
